File: HW2/PCB Design/Lu_hw2.brd (EAGLE design)
At the start: 50 x 50 mm, 22 parts, among them J2 USB-MB-H

Commit message: edit
Parts:
- removed LED2: (no value), Lu_hw2:LED3MM
- removed R2: 330, Lu_hw2:0207/10
- removed USER_BUTTON: (no value), Lu_hw2:1X03
- added LED3: (no value), Lu_hw2:LED3MM
- added R4: 330, Lu_hw2:0207/10
- added USER_BUTTON1: (no value), Lu_hw2:1X03
- moved J2 38.1 mm to (6.35, 44.5), turned to 270 degrees
- moved C7 25.4 mm to (35.6, 6.35)
- moved C5 17.8 mm to (35.6, 24.1)
- moved C2 14.0 mm to (14.0, 22.9)
- moved R3 14.0 mm to (14.0, 36.8)
- moved LED1 12.0 mm to (10.2, 33.0)
- moved J5 11.4 mm to (3.81, 34.3)
- moved U$3 10.9 mm to (36.8, 38.1), turned to 270 degrees
- moved U$1 9.67 mm to (30.5, 47.0), turned to 180 degrees
- moved C3 8.13 mm to (41.9, 24.1)
- moved RESET_BUTTON 7.62 mm to (47.0, 31.8)
- moved C6 6.35 mm to (35.6, 19.1)
- moved C8 5.68 mm to (38.1, 30.5)
- moved R1 5.68 mm to (14.0, 26.7), turned to 180 degrees
- moved RESONATOR 4.02 mm to (11.4, 17.8)
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Connections:
- removed net N$7: LED2.K, R2.2
- new net N$4: LED3.A, R4.2
- net A4: now also R4.1; no longer LED2.A
- net B4: no longer USER_BUTTON.3
- net GND: now also LED3.K, USER_BUTTON1.1; no longer R2.1, USER_BUTTON.1

Commit message: edit
Parts:
- removed LED3: (no value), Lu_hw2:LED3MM
- removed R5: 10K, Lu_hw2:0207/10
- added LED2: (no value), Lu_hw2:LED3MM
- added R2: 10K, Lu_hw2:0207/10
- moved USER_BUTTON1 27.5 mm to (17.8, 8.89), turned to 90 degrees
- moved C2 21.7 mm to (16.5, 44.5)
- moved R1 16.5 mm to (7.62, 11.4), turned to 90 degrees
- moved R4 16.5 mm to (12.7, 6.35), turned to 270 degrees
- moved J2 15.2 mm to (6.35, 29.2), turned to 0 degrees
- moved J5 11.4 mm to (3.81, 45.7)
- moved RESONATOR 6.48 mm to (17.8, 16.5), turned to 90 degrees
- moved LED1 6.48 mm to (8.89, 39.4)
- moved C6 5.68 mm to (40.6, 16.5)
- moved C8 5.08 mm to (43.2, 30.5)
- moved R3 4.58 mm to (17.8, 34.3), turned to 90 degrees
- moved C5 2.54 mm to (35.6, 21.6)
- moved RESET_BUTTON 2.54 mm to (47.0, 34.3)
- moved U$1 2.54 mm to (30.5, 44.5)
- moved C3 1.27 mm to (43.2, 24.1)
Connections:
- net +3V3: now also R2.2; no longer R5.1
- net B4: now also R2.1, USER_BUTTON1.3; no longer R5.2
- net GND: now also LED2.K; no longer LED3.K
- net N$4: now also LED2.A; no longer LED3.A

Commit message: edit
Routing:
- net +5V: track 0.00 -> 60.0 mm
- net MCLR: track 0.00 -> 29.2 mm
- net B14: track 0.00 -> 25.3 mm, vias 0 -> 1
- net +3V3: track 0.00 -> 25.2 mm, vias 0 -> 1
- net B13: track 0.00 -> 23.8 mm, vias 0 -> 1
- net B9: track 0.00 -> 17.8 mm
- net B8: track 0.00 -> 17.8 mm
- net B7: track 0.00 -> 17.8 mm
- net N$10: track 0.00 -> 13.8 mm
Changed lines of the file:
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@@
 <contactref element="J3" pad="1"/>
 <contactref element="U$3" pad="P$1"/>
-<polygon width="0.4064" layer="16" isolate="0.012">
+<polygon width="0.4064" layer="16" isolate="0.3048">
 <vertex x="0" y="49.53"/>
 <vertex x="49.53" y="49.53"/>
@@
 <contactref element="J1" pad="2"/>
 <contactref element="R2" pad="2"/>
+<wire x1="41.91" y1="30.48" x2="41.91" y2="24.13" width="0.4064" layer="1"/>
+<wire x1="41.91" y1="24.13" x2="40.64" y2="24.13" width="0.4064" layer="16"/>
+<wire x1="40.64" y1="24.13" x2="40.64" y2="22.86" width="0.4064" layer="16"/>
+<wire x1="40.64" y1="22.86" x2="39.37" y2="21.59" width="0.4064" layer="16"/>
+<wire x1="39.37" y1="21.59" x2="36.83" y2="21.59" width="0.4064" layer="16"/>
+<wire x1="29.21" y1="26.67" x2="35.56" y2="26.67" width="0.4064" layer="16"/>
+<via x="35.56" y="26.67" extent="1-16" drill="0.6" shape="square"/>
+<wire x1="35.56" y1="26.67" x2="35.56" y2="22.86" width="0.4064" layer="1"/>
+<wire x1="35.56" y1="22.86" x2="36.83" y2="21.59" width="0.4064" layer="1"/>
 <wire x1="29.21" y1="39.37" x2="29.21" y2="44.45" width="0" layer="19" extent="1-1"/>
 <wire x1="29.21" y1="26.67" x2="29.21" y2="39.37" width="0" layer="19" extent="1-1"/>
-<wire x1="36.83" y1="21.59" x2="29.21" y2="26.67" width="0" layer="19" extent="1-1"/>
-<wire x1="41.91" y1="24.13" x2="36.83" y2="21.59" width="0" layer="19" extent="1-1"/>
-<wire x1="41.91" y1="30.48" x2="41.91" y2="24.13" width="0" layer="19" extent="1-1"/>
 <wire x1="17.78" y1="29.21" x2="29.21" y2="26.67" width="0" layer="19" extent="1-1"/>
 <wire x1="7.62" y1="6.35" x2="17.78" y2="29.21" width="0" layer="19" extent="1-1"/>
@@
 <contactref element="U$2" pad="1"/>
 <contactref element="J5" pad="1"/>
-<wire x1="21.59" y1="39.37" x2="46.99" y2="39.37" width="0" layer="19" extent="1-1"/>
+<wire x1="17.78" y1="39.37" x2="46.99" y2="39.37" width="0.4064" layer="16"/>
 <wire x1="17.78" y1="39.37" x2="21.59" y2="39.37" width="0" layer="19" extent="1-1"/>
 <wire x1="3.81" y1="45.72" x2="17.78" y2="39.37" width="0" layer="19" extent="1-1"/>
@@
 <contactref element="U$2" pad="20"/>
 <contactref element="C6" pad="+"/>
-<wire x1="29.21" y1="19.05" x2="41.91" y2="16.51" width="0" layer="19" extent="1-1"/>
+<wire x1="29.21" y1="19.05" x2="39.37" y2="19.05" width="0.4064" layer="16"/>
+<wire x1="39.37" y1="19.05" x2="41.91" y2="16.51" width="0.4064" layer="16"/>
 </signal>
 <signal name="D+">
@@
 <contactref element="U$2" pad="25"/>
 <contactref element="J3" pad="7"/>
-<wire x1="29.21" y1="31.75" x2="46.99" y2="19.05" width="0" layer="19" extent="1-1"/>
+<wire x1="46.99" y1="19.05" x2="45.72" y2="19.05" width="0.4064" layer="1"/>
+<wire x1="45.72" y1="19.05" x2="38.1" y2="26.67" width="0.4064" layer="1"/>
+<wire x1="38.1" y1="26.67" x2="38.1" y2="30.48" width="0.4064" layer="1"/>
+<wire x1="38.1" y1="30.48" x2="36.83" y2="31.75" width="0.4064" layer="1"/>
+<via x="36.83" y="31.75" extent="1-16" drill="0.6" shape="square"/>
+<wire x1="36.83" y1="31.75" x2="29.21" y2="31.75" width="0.4064" layer="16"/>
 </signal>
 <signal name="B13">
 <contactref element="U$2" pad="24"/>
 <contactref element="J3" pad="6"/>
-<wire x1="29.21" y1="29.21" x2="46.99" y2="16.51" width="0" layer="19" extent="1-1"/>
+<wire x1="29.21" y1="29.21" x2="35.56" y2="29.21" width="0.4064" layer="16"/>
+<wire x1="35.56" y1="29.21" x2="36.83" y2="27.94" width="0.4064" layer="16"/>
+<via x="36.83" y="27.94" extent="1-16" drill="0.6" shape="square"/>
+<wire x1="36.83" y1="27.94" x2="36.83" y2="26.67" width="0.4064" layer="1"/>
+<wire x1="36.83" y1="26.67" x2="46.99" y2="16.51" width="0.4064" layer="1"/>
 </signal>
 <signal name="B9">
 <contactref element="U$2" pad="18"/>
 <contactref element="J3" pad="5"/>
-<wire x1="29.21" y1="13.97" x2="46.99" y2="13.97" width="0" layer="19" extent="1-1"/>
+<wire x1="29.21" y1="13.97" x2="46.99" y2="13.97" width="0.4064" layer="16"/>
 </signal>
 <signal name="B8">
 <contactref element="U$2" pad="17"/>
 <contactref element="J3" pad="4"/>
-<wire x1="29.21" y1="11.43" x2="46.99" y2="11.43" width="0" layer="19" extent="1-1"/>
+<wire x1="29.21" y1="11.43" x2="46.99" y2="11.43" width="0.4064" layer="16"/>
 </signal>
 <signal name="B7">
 <contactref element="U$2" pad="16"/>
 <contactref element="J3" pad="3"/>
-<wire x1="29.21" y1="8.89" x2="46.99" y2="8.89" width="0" layer="19" extent="1-1"/>
+<wire x1="29.21" y1="8.89" x2="46.99" y2="8.89" width="0.4064" layer="16"/>
 </signal>
 <signal name="+5V">
@@
 <contactref element="U$2" pad="15"/>
 <contactref element="U$3" pad="P$3"/>
-<wire x1="34.83" y1="37.1" x2="30.48" y2="42.545" width="0" layer="19" extent="1-1"/>
-<wire x1="34.29" y1="6.35" x2="34.83" y2="37.1" width="0" layer="19" extent="1-1"/>
-<wire x1="29.21" y1="6.35" x2="34.29" y2="6.35" width="0" layer="19" extent="1-1"/>
-<wire x1="46.99" y1="6.35" x2="34.29" y2="6.35" width="0" layer="19" extent="1-1"/>
+<wire x1="46.99" y1="6.35" x2="44.45" y2="6.35" width="0.4064" layer="16"/>
+<wire x1="44.45" y1="6.35" x2="41.91" y2="3.81" width="0.4064" layer="16"/>
+<wire x1="41.91" y1="3.81" x2="36.83" y2="3.81" width="0.4064" layer="16"/>
+<wire x1="36.83" y1="3.81" x2="34.29" y2="6.35" width="0.4064" layer="16"/>
+<wire x1="29.21" y1="6.35" x2="34.29" y2="6.35" width="0.4064" layer="16"/>
+<wire x1="34.29" y1="6.35" x2="34.29" y2="36.56" width="0.4064" layer="1"/>
+<wire x1="34.29" y1="36.56" x2="34.83" y2="37.1" width="0.4064" layer="1"/>
+<wire x1="30.48" y1="42.545" x2="33.655" y2="42.545" width="0.4064" layer="1"/>
+<wire x1="33.655" y1="42.545" x2="34.29" y2="41.91" width="0.4064" layer="1"/>
+<wire x1="34.29" y1="41.91" x2="34.29" y2="37.64" width="0.4064" layer="1"/>
+<wire x1="34.29" y1="37.64" x2="34.83" y2="37.1" width="0.4064" layer="1"/>
 </signal>
 <signal name="N$1">

Commit message: edit
Parts:
- moved R2 1.27 mm to (10.2, 8.89)
Routing:
- net B15: track 0.00 -> 28.2 mm, vias 0 -> 1
- net +3V3: track 25.2 -> 53.2 mm
- net MCLR: track 29.2 -> 52.2 mm, vias 0 -> 2
- net VSS: track 0.00 -> 15.5 mm
- net VDD: track 0.00 -> 14.1 mm, vias 0 -> 3
- net N$4: track 0.00 -> 4.86 mm
Changed lines of the file:
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@@
 <element name="R4" library="Lu_hw2" package="0207/10" value="330" x="12.7" y="6.35" rot="R270"/>
 <element name="USER_BUTTON1" library="Lu_hw2" package="1X03" value="" x="17.78" y="8.89" rot="R90"/>
-<element name="R2" library="Lu_hw2" package="0207/10" value="10K" x="10.16" y="7.62" rot="R270"/>
+<element name="R2" library="Lu_hw2" package="0207/10" value="10K" x="10.16" y="8.89" rot="R270"/>
 </elements>
 <signals>
@@
 <wire x1="35.56" y1="26.67" x2="35.56" y2="22.86" width="0.4064" layer="1"/>
 <wire x1="35.56" y1="22.86" x2="36.83" y2="21.59" width="0.4064" layer="1"/>
-<wire x1="29.21" y1="39.37" x2="29.21" y2="44.45" width="0" layer="19" extent="1-1"/>
-<wire x1="29.21" y1="26.67" x2="29.21" y2="39.37" width="0" layer="19" extent="1-1"/>
-<wire x1="17.78" y1="29.21" x2="29.21" y2="26.67" width="0" layer="19" extent="1-1"/>
+<wire x1="29.21" y1="44.45" x2="29.21" y2="39.37" width="0.4064" layer="1"/>
+<wire x1="29.21" y1="26.67" x2="27.94" y2="26.67" width="0.4064" layer="1"/>
+<wire x1="27.94" y1="26.67" x2="26.67" y2="27.94" width="0.4064" layer="1"/>
+<wire x1="26.67" y1="27.94" x2="26.67" y2="36.83" width="0.4064" layer="1"/>
+<wire x1="26.67" y1="36.83" x2="29.21" y2="39.37" width="0.4064" layer="1"/>
+<wire x1="10.16" y1="3.81" x2="7.62" y2="6.35" width="0.4064" layer="1"/>
+<wire x1="3.81" y1="6.35" x2="7.62" y2="6.35" width="0.4064" layer="16"/>
+<wire x1="17.78" y1="29.21" x2="26.67" y2="27.94" width="0" layer="19" extent="1-1"/>
 <wire x1="7.62" y1="6.35" x2="17.78" y2="29.21" width="0" layer="19" extent="1-1"/>
-<wire x1="3.81" y1="6.35" x2="7.62" y2="6.35" width="0" layer="19" extent="1-1"/>
-<wire x1="10.16" y1="2.54" x2="7.62" y2="6.35" width="0" layer="19" extent="1-1"/>
 </signal>
 <signal name="MCLR">
@@
 <contactref element="U$2" pad="1"/>
 <contactref element="J5" pad="1"/>
-<wire x1="17.78" y1="39.37" x2="46.99" y2="39.37" width="0.4064" layer="16"/>
-<wire x1="17.78" y1="39.37" x2="21.59" y2="39.37" width="0" layer="19" extent="1-1"/>
-<wire x1="3.81" y1="45.72" x2="17.78" y2="39.37" width="0" layer="19" extent="1-1"/>
+<wire x1="17.78" y1="39.37" x2="21.59" y2="39.37" width="0.4064" layer="16"/>
+<wire x1="46.99" y1="39.37" x2="45.72" y2="39.37" width="0.4064" layer="16"/>
+<wire x1="45.72" y1="39.37" x2="44.45" y2="40.64" width="0.4064" layer="16"/>
+<wire x1="44.45" y1="40.64" x2="19.05" y2="40.64" width="0.4064" layer="16"/>
+<wire x1="19.05" y1="40.64" x2="17.78" y2="39.37" width="0.4064" layer="16"/>
+<wire x1="3.81" y1="45.72" x2="10.16" y2="45.72" width="0.4064" layer="16"/>
+<wire x1="10.16" y1="45.72" x2="11.43" y2="44.45" width="0.4064" layer="16"/>
+<via x="11.43" y="44.45" extent="1-16" drill="0.6" shape="square"/>
+<wire x1="11.43" y1="44.45" x2="11.43" y2="41.91" width="0.4064" layer="1"/>
+<wire x1="11.43" y1="41.91" x2="13.97" y2="39.37" width="0.4064" layer="1"/>
+<via x="13.97" y="39.37" extent="1-16" drill="0.6" shape="square"/>
+<wire x1="13.97" y1="39.37" x2="17.78" y2="39.37" width="0.4064" layer="16"/>
 </signal>
 <signal name="N$2">
@@
 <contactref element="U$2" pad="13"/>
 <contactref element="J5" pad="2"/>
-<wire x1="3.81" y1="43.18" x2="15.24" y2="44.45" width="0" layer="19" extent="1-1"/>
+<wire x1="3.81" y1="43.18" x2="7.62" y2="43.18" width="0.4064" layer="16"/>
+<via x="7.62" y="43.18" extent="1-16" drill="0.6" shape="square"/>
+<wire x1="7.62" y1="43.18" x2="11.43" y2="46.99" width="0.4064" layer="1"/>
+<via x="11.43" y="46.99" extent="1-16" drill="0.6" shape="square"/>
+<wire x1="11.43" y1="46.99" x2="12.7" y2="46.99" width="0.4064" layer="16"/>
+<via x="12.7" y="46.99" extent="1-16" drill="0.6" shape="square"/>
+<wire x1="12.7" y1="46.99" x2="15.24" y2="44.45" width="0.4064" layer="1"/>
 <wire x1="21.59" y1="8.89" x2="15.24" y2="44.45" width="0" layer="19" extent="1-1"/>
 </signal>
@@
 <contactref element="C2" pad="1"/>
 <contactref element="J5" pad="3"/>
-<wire x1="3.81" y1="40.64" x2="17.78" y2="44.45" width="0" layer="19" extent="1-1"/>
-<wire x1="21.59" y1="21.59" x2="17.78" y2="44.45" width="0" layer="19" extent="1-1"/>
+<wire x1="3.81" y1="40.64" x2="8.89" y2="40.64" width="0.4064" layer="16"/>
+<wire x1="8.89" y1="40.64" x2="10.16" y2="41.91" width="0.4064" layer="16"/>
+<wire x1="10.16" y1="41.91" x2="15.24" y2="41.91" width="0.4064" layer="16"/>
+<wire x1="15.24" y1="41.91" x2="17.78" y2="44.45" width="0.4064" layer="16"/>
+<wire x1="21.59" y1="21.59" x2="15.24" y2="41.91" width="0" layer="19" extent="16-16"/>
 </signal>
 <signal name="PGD1">
@@
 <contactref element="R2" pad="1"/>
 <wire x1="17.78" y1="13.97" x2="21.59" y2="13.97" width="0" layer="19" extent="1-1"/>
-<wire x1="10.16" y1="12.7" x2="17.78" y2="13.97" width="0" layer="19" extent="1-1"/>
-<wire x1="3.81" y1="11.43" x2="10.16" y2="12.7" width="0" layer="19" extent="1-1"/>
+<wire x1="10.16" y1="13.97" x2="17.78" y2="13.97" width="0" layer="19" extent="1-1"/>
+<wire x1="3.81" y1="11.43" x2="10.16" y2="13.97" width="0" layer="19" extent="1-1"/>
 </signal>
 <signal name="A4">
@@
 <contactref element="U$2" pad="26"/>
 <contactref element="J3" pad="8"/>
-<wire x1="29.21" y1="34.29" x2="46.99" y2="21.59" width="0" layer="19" extent="1-1"/>
+<wire x1="46.99" y1="21.59" x2="46.99" y2="30.48" width="0.4064" layer="1"/>
+<wire x1="46.99" y1="30.48" x2="43.18" y2="34.29" width="0.4064" layer="1"/>
+<via x="43.18" y="34.29" extent="1-16" drill="0.6" shape="square"/>
+<wire x1="43.18" y1="34.29" x2="29.21" y2="34.29" width="0.4064" layer="16"/>
 </signal>
 <signal name="B14">
@@
 <contactref element="LED2" pad="A"/>
 <contactref element="R4" pad="2"/>
-<wire x1="12.7" y1="1.27" x2="16.51" y2="3.81" width="0" layer="19" extent="1-1"/>
+<wire x1="12.7" y1="1.27" x2="13.97" y2="1.27" width="0.4064" layer="1"/>
+<wire x1="13.97" y1="1.27" x2="16.51" y2="3.81" width="0.4064" layer="1"/>
 </signal>
 </signals>

Commit message: edit
Routing:
- net +3V3: track 53.2 -> 93.0 mm, vias 1 -> 5
- net A4: track 0.00 -> 28.0 mm, vias 0 -> 1
- net N$2: track 0.00 -> 23.9 mm
- net B4: track 0.00 -> 18.8 mm
- net N$3: track 0.00 -> 4.86 mm
- net N$5: track 0.00 -> 3.81 mm
Changed lines of the file:
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@@
 <wire x1="10.16" y1="3.81" x2="7.62" y2="6.35" width="0.4064" layer="1"/>
 <wire x1="3.81" y1="6.35" x2="7.62" y2="6.35" width="0.4064" layer="16"/>
-<wire x1="17.78" y1="29.21" x2="26.67" y2="27.94" width="0" layer="19" extent="1-1"/>
-<wire x1="7.62" y1="6.35" x2="17.78" y2="29.21" width="0" layer="19" extent="1-1"/>
+<wire x1="7.62" y1="6.35" x2="7.62" y2="13.97" width="0.4064" layer="1"/>
+<wire x1="7.62" y1="13.97" x2="10.16" y2="16.51" width="0.4064" layer="1"/>
+<via x="10.16" y="16.51" extent="1-16" drill="0.6" shape="square"/>
+<wire x1="10.16" y1="16.51" x2="13.97" y2="16.51" width="0.4064" layer="16"/>
+<via x="13.97" y="16.51" extent="1-16" drill="0.6" shape="square"/>
+<wire x1="13.97" y1="16.51" x2="15.24" y2="17.78" width="0.4064" layer="1"/>
+<wire x1="15.24" y1="17.78" x2="15.24" y2="26.67" width="0.4064" layer="1"/>
+<wire x1="15.24" y1="26.67" x2="17.78" y2="29.21" width="0.4064" layer="1"/>
+<wire x1="17.78" y1="29.21" x2="19.05" y2="29.21" width="0.4064" layer="1"/>
+<wire x1="19.05" y1="29.21" x2="20.32" y2="30.48" width="0.4064" layer="1"/>
+<via x="20.32" y="30.48" extent="1-16" drill="0.6" shape="square"/>
+<wire x1="20.32" y1="30.48" x2="24.13" y2="30.48" width="0.4064" layer="16"/>
+<via x="24.13" y="30.48" extent="1-16" drill="0.6" shape="square"/>
+<wire x1="24.13" y1="30.48" x2="26.67" y2="27.94" width="0.4064" layer="1"/>
 </signal>
 <signal name="MCLR">
@@
 <contactref element="LED1" pad="A"/>
 <contactref element="R1" pad="2"/>
-<wire x1="7.62" y1="16.51" x2="7.62" y2="39.37" width="0" layer="19" extent="1-1"/>
+<wire x1="7.62" y1="16.51" x2="7.62" y2="22.86" width="0.4064" layer="1"/>
+<wire x1="7.62" y1="22.86" x2="8.89" y2="24.13" width="0.4064" layer="1"/>
+<wire x1="8.89" y1="24.13" x2="8.89" y2="38.1" width="0.4064" layer="1"/>
+<wire x1="8.89" y1="38.1" x2="7.62" y2="39.37" width="0.4064" layer="1"/>
 </signal>
 <signal name="N$3">
 <contactref element="U$2" pad="9"/>
 <contactref element="RESONATOR" pad="3"/>
-<wire x1="17.78" y1="21.59" x2="21.59" y2="19.05" width="0" layer="19" extent="1-1"/>
+<wire x1="21.59" y1="19.05" x2="20.32" y2="19.05" width="0.4064" layer="1"/>
+<wire x1="20.32" y1="19.05" x2="17.78" y2="21.59" width="0.4064" layer="1"/>
 </signal>
 <signal name="N$5">
 <contactref element="U$2" pad="10"/>
 <contactref element="RESONATOR" pad="1"/>
-<wire x1="17.78" y1="16.51" x2="21.59" y2="16.51" width="0" layer="19" extent="1-1"/>
+<wire x1="17.78" y1="16.51" x2="21.59" y2="16.51" width="0.4064" layer="16"/>
 </signal>
 <signal name="N$10">
@@
 <contactref element="USER_BUTTON1" pad="3"/>
 <contactref element="R2" pad="1"/>
-<wire x1="17.78" y1="13.97" x2="21.59" y2="13.97" width="0" layer="19" extent="1-1"/>
-<wire x1="10.16" y1="13.97" x2="17.78" y2="13.97" width="0" layer="19" extent="1-1"/>
-<wire x1="3.81" y1="11.43" x2="10.16" y2="13.97" width="0" layer="19" extent="1-1"/>
+<wire x1="3.81" y1="11.43" x2="7.62" y2="11.43" width="0.4064" layer="16"/>
+<wire x1="7.62" y1="11.43" x2="10.16" y2="13.97" width="0.4064" layer="16"/>
+<wire x1="10.16" y1="13.97" x2="17.78" y2="13.97" width="0.4064" layer="16"/>
+<wire x1="21.59" y1="13.97" x2="17.78" y2="13.97" width="0.4064" layer="16"/>
 </signal>
 <signal name="A4">
@@
 <contactref element="R4" pad="1"/>
 <contactref element="U$2" pad="12"/>
-<wire x1="12.7" y1="11.43" x2="21.59" y2="11.43" width="0" layer="19" extent="1-1"/>
-<wire x1="3.81" y1="8.89" x2="12.7" y2="11.43" width="0" layer="19" extent="1-1"/>
+<wire x1="12.7" y1="11.43" x2="12.7" y2="10.16" width="0.4064" layer="16"/>
+<wire x1="24.13" y1="10.16" x2="24.13" y2="8.89" width="0.4064" layer="1"/>
+<wire x1="24.13" y1="8.89" x2="22.86" y2="7.62" width="0.4064" layer="1"/>
+<via x="22.86" y="7.62" extent="1-16" drill="0.6" shape="square"/>
+<wire x1="22.86" y1="7.62" x2="15.24" y2="7.62" width="0.4064" layer="16"/>
+<wire x1="15.24" y1="7.62" x2="12.7" y2="10.16" width="0.4064" layer="16"/>
+<wire x1="3.81" y1="8.89" x2="11.43" y2="8.89" width="0.4064" layer="16"/>
+<wire x1="11.43" y1="8.89" x2="12.7" y2="10.16" width="0.4064" layer="16"/>
+<wire x1="21.59" y1="11.43" x2="22.86" y2="11.43" width="0.4064" layer="1"/>
+<wire x1="22.86" y1="11.43" x2="24.13" y2="10.16" width="0.4064" layer="1"/>
 </signal>
 <signal name="A0">

Commit message: edit
Parts:
- moved J5 1.27 mm to (5.08, 45.7)
- moved LED1 1.27 mm to (10.2, 39.4)
Routing:
- net VDD: track 14.1 -> 63.7 mm, vias 3 -> 7
- net N$1: track 0.00 -> 46.8 mm, vias 0 -> 2
- net D-: track 0.00 -> 43.8 mm, vias 0 -> 2
- net VSS: track 15.5 -> 54.8 mm, vias 0 -> 3
- net A0: track 0.00 -> 28.1 mm, vias 0 -> 2
- net B3: track 0.00 -> 26.5 mm, vias 0 -> 3
- net A1: track 0.00 -> 25.6 mm, vias 0 -> 2
- net B2: track 0.00 -> 25.0 mm, vias 0 -> 3
- net D+: track 0.00 -> 23.9 mm, vias 0 -> 2
- net PGD1: track 0.00 -> 19.1 mm
- net PGC1: track 0.00 -> 19.1 mm
- net MCLR: track 52.2 -> 50.9 mm
- net N$2: track 23.9 -> 23.4 mm

Commit message: edit
Parts:
- U$3: value SWITCH -> (none)
- moved U$3 1.27 mm to (38.1, 38.1)
- renumbered RESET_BUTTON to RESET, USER_BUTTON1 to USER
Connections:
- net +5V: now also U$3.3.VOUT; no longer U$3.P$3
- net GND: now also U$3.1.GND; no longer U$3.P$1
- net N$1: now also U$3.2.VIN; no longer U$3.P$2
Routing:
- net +5V: track 60.0 -> 66.9 mm
- net N$1: track 46.8 -> 49.5 mm
Other:
- board text added: "10K"
- board text added: "330"
- board text added: "3V3"
- board text added: "A0"
- board text added: "A1"
- board text added: "A4"
- board text added: "B2"
- board text added: "B3"
- board text added: "B4"
- board text added: "GND"
- board text added: "MCLR"
- board text added: "PGC1"
- board text added: "PGD1"
- board text added: "VDD"
- board text added: "VIN"
- board text added: "VOUT"
