File: HW2/PCB Design/Lu_hw2.brd (EAGLE design)
At the start: 50 x 50 mm, 22 parts, among them J2 USB-MB-H

Commit message: error check
Routing:
- net +3V3: track 93.0 -> 91.0 mm
- net D-: track 43.8 -> 42.0 mm, vias 2 -> 3
- net A4: track 28.0 -> 29.1 mm
- net B14: track 25.3 -> 26.0 mm
- net B13: track 23.8 -> 24.5 mm
- net VDD: vias 7 -> 5
Other:
- board text added: "D+"
- board text added: "D-"
- board text added: "Li-Chun (David) Lu April 2016"
- board text added: "MECH 433 Advanced Mechatronics"
- board text added: "Northwestern University"
