File: HW2/PCB Design/Lu_hw2.brd (EAGLE design)
At the start: 50 x 50 mm, 22 parts, among them J2 USB-MB-H

Commit message: edit
Parts:
- renumbered RESONATOR to 8MHZ
Connections:
- new net B5: J2.ID, U$2.14
Routing:
- net B5: track 0.00 -> 30.5 mm
Changed lines of the file:
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@@
 <layer number="27" name="tValues" color="7" fill="1" visible="yes" active="yes"/>
 <layer number="28" name="bValues" color="7" fill="1" visible="yes" active="yes"/>
-<layer number="29" name="tStop" color="7" fill="3" visible="no" active="yes"/>
-<layer number="30" name="bStop" color="7" fill="6" visible="no" active="yes"/>
-<layer number="31" name="tCream" color="7" fill="4" visible="no" active="yes"/>
-<layer number="32" name="bCream" color="7" fill="5" visible="no" active="yes"/>
-<layer number="33" name="tFinish" color="6" fill="3" visible="no" active="yes"/>
-<layer number="34" name="bFinish" color="6" fill="6" visible="no" active="yes"/>
-<layer number="35" name="tGlue" color="7" fill="4" visible="no" active="yes"/>
-<layer number="36" name="bGlue" color="7" fill="5" visible="no" active="yes"/>
-<layer number="37" name="tTest" color="7" fill="1" visible="no" active="yes"/>
-<layer number="38" name="bTest" color="7" fill="1" visible="no" active="yes"/>
+<layer number="29" name="tStop" color="7" fill="3" visible="yes" active="yes"/>
+<layer number="30" name="bStop" color="7" fill="6" visible="yes" active="yes"/>
+<layer number="31" name="tCream" color="7" fill="4" visible="yes" active="yes"/>
+<layer number="32" name="bCream" color="7" fill="5" visible="yes" active="yes"/>
+<layer number="33" name="tFinish" color="6" fill="3" visible="yes" active="yes"/>
+<layer number="34" name="bFinish" color="6" fill="6" visible="yes" active="yes"/>
+<layer number="35" name="tGlue" color="7" fill="4" visible="yes" active="yes"/>
+<layer number="36" name="bGlue" color="7" fill="5" visible="yes" active="yes"/>
+<layer number="37" name="tTest" color="7" fill="1" visible="yes" active="yes"/>
+<layer number="38" name="bTest" color="7" fill="1" visible="yes" active="yes"/>
 <layer number="39" name="tKeepout" color="4" fill="11" visible="yes" active="yes"/>
 <layer number="40" name="bKeepout" color="1" fill="11" visible="yes" active="yes"/>
@@
 <layer number="42" name="bRestrict" color="1" fill="10" visible="yes" active="yes"/>
 <layer number="43" name="vRestrict" color="2" fill="10" visible="yes" active="yes"/>
-<layer number="44" name="Drills" color="7" fill="1" visible="no" active="yes"/>
-<layer number="45" name="Holes" color="7" fill="1" visible="no" active="yes"/>
-<layer number="46" name="Milling" color="3" fill="1" visible="no" active="yes"/>
-<layer number="47" name="Measures" color="7" fill="1" visible="no" active="yes"/>
+<layer number="44" name="Drills" color="7" fill="1" visible="yes" active="yes"/>
+<layer number="45" name="Holes" color="7" fill="1" visible="yes" active="yes"/>
+<layer number="46" name="Milling" color="3" fill="1" visible="yes" active="yes"/>
+<layer number="47" name="Measures" color="7" fill="1" visible="yes" active="yes"/>
 <layer number="48" name="Document" color="7" fill="1" visible="yes" active="yes"/>
 <layer number="49" name="Reference" color="7" fill="1" visible="yes" active="yes"/>
@@
 <attribute name="VALUE" x="50.165" y="33.02" size="1.27" layer="27" rot="R90"/>
 </element>
-<element name="RESONATOR" library="Lu_hw2" package="1X03" value="" x="17.78" y="16.51" smashed="yes" rot="R90">
+<element name="8MHZ" library="Lu_hw2" package="1X03" value="" x="17.78" y="16.51" smashed="yes" rot="R90">
 <attribute name="NAME" x="15.9512" y="15.1638" size="0.8128" layer="25" ratio="10" rot="R90"/>
 <attribute name="VALUE" x="20.955" y="15.24" size="1.27" layer="27" rot="R90"/>
@@
 <contactref element="U$2" pad="27"/>
 <contactref element="C3" pad="2"/>
-<contactref element="RESONATOR" pad="2"/>
+<contactref element="8MHZ" pad="2"/>
 <contactref element="J1" pad="1"/>
 <contactref element="J3" pad="1"/>
@@
 <signal name="N$3">
 <contactref element="U$2" pad="9"/>
-<contactref element="RESONATOR" pad="3"/>
+<contactref element="8MHZ" pad="3"/>
 <wire x1="21.59" y1="19.05" x2="20.32" y2="19.05" width="0.4064" layer="1"/>
 <wire x1="20.32" y1="19.05" x2="17.78" y2="21.59" width="0.4064" layer="1"/>
@@
 <signal name="N$5">
 <contactref element="U$2" pad="10"/>
-<contactref element="RESONATOR" pad="1"/>
+<contactref element="8MHZ" pad="1"/>
 <wire x1="17.78" y1="16.51" x2="21.59" y2="16.51" width="0.4064" layer="16"/>
 </signal>
@@
 <wire x1="13.97" y1="1.27" x2="16.51" y2="3.81" width="0.4064" layer="1"/>
 </signal>
+<signal name="B5">
+<contactref element="U$2" pad="14"/>
+<contactref element="J2" pad="ID"/>
+<wire x1="10.25" y1="28.41" x2="10.25" y2="18.325" width="0.4064" layer="1"/>
+<wire x1="10.25" y1="18.325" x2="12.7" y2="15.875" width="0.4064" layer="1"/>
+<wire x1="12.7" y1="15.875" x2="12.7" y2="13.97" width="0.4064" layer="1"/>
+<wire x1="12.7" y1="13.97" x2="15.24" y2="11.43" width="0.4064" layer="1"/>
+<wire x1="15.24" y1="11.43" x2="15.24" y2="6.35" width="0.4064" layer="1"/>
+<wire x1="15.24" y1="6.35" x2="21.59" y2="6.35" width="0.4064" layer="1"/>
+</signal>
 </signals>
