File: HW2/PCB Design/Lu_hw2.sch (EAGLE design)
At the start: 22 parts, among them J2 USB-MB-H

Commit message: edit
Parts:
- removed LED2: (no value), Lu_hw2:LED3MM
- removed R2: 330, Lu_hw2:R-US_0207/10
- removed USER_BUTTON: (no value), Lu_hw2:M03PTH
- added LED3: (no value), Lu_hw2:LED3MM
- added R4: 330, Lu_hw2:R-US_0207/10
- added USER_BUTTON1: (no value), Lu_hw2:M03PTH
Connections:
- removed net N$7: LED2.C, R2.2
- new net N$4: LED3.A, R4.2
- net A4: now also R4.1; no longer LED2.A
- net B4: no longer USER_BUTTON.3
- net GND: now also LED3.C, USER_BUTTON1.1; no longer R2.1, USER_BUTTON.1
Changed lines of the file:
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@@
 <part name="U$1" library="Lu_hw2" deviceset="MCP1702" device=""/>
 <part name="LED1" library="Lu_hw2" deviceset="LED" device="3MM"/>
-<part name="LED2" library="Lu_hw2" deviceset="LED" device="3MM"/>
 <part name="R1" library="Lu_hw2" deviceset="R-US_" device="0207/10" value="330"/>
-<part name="R2" library="Lu_hw2" deviceset="R-US_" device="0207/10" value="330"/>
 <part name="R3" library="Lu_hw2" deviceset="R-US_" device="0207/10" value="10K"/>
 <part name="C2" library="Lu_hw2" deviceset="C-US" device="025-030X050" value="0.1uF"/>
@@
 <part name="+3V10" library="Lu_hw2" deviceset="+3V3" device=""/>
 <part name="GND14" library="Lu_hw2" deviceset="GND" device=""/>
-<part name="GND15" library="Lu_hw2" deviceset="GND" device=""/>
-<part name="USER_BUTTON" library="Lu_hw2" deviceset="M03" device="PTH"/>
-<part name="GND3" library="Lu_hw2" deviceset="GND" device=""/>
 <part name="RESET_BUTTON" library="Lu_hw2" deviceset="M03" device="PTH"/>
 <part name="GND4" library="Lu_hw2" deviceset="GND" device=""/>
@@
 <part name="U$3" library="Lu_hw2" deviceset="SWITCH" device=""/>
 <part name="GND8" library="Lu_hw2" deviceset="GND" device=""/>
+<part name="LED3" library="Lu_hw2" deviceset="LED" device="3MM"/>
+<part name="GND16" library="Lu_hw2" deviceset="GND" device=""/>
+<part name="R4" library="Lu_hw2" deviceset="R-US_" device="0207/10" value="330"/>
+<part name="USER_BUTTON1" library="Lu_hw2" deviceset="M03" device="PTH"/>
+<part name="GND15" library="Lu_hw2" deviceset="GND" device=""/>
 </parts>
 <sheets>
@@
 <instance part="U$1" gate="G$1" x="-48.26" y="137.16" rot="R90"/>
 <instance part="LED1" gate="G$1" x="-99.06" y="96.52" rot="R90"/>
-<instance part="LED2" gate="G$1" x="-99.06" y="30.48" rot="R270"/>
 <instance part="R1" gate="G$1" x="-109.22" y="96.52"/>
-<instance part="R2" gate="G$1" x="-111.76" y="30.48"/>
 <instance part="R3" gate="G$1" x="-104.14" y="86.36"/>
 <instance part="C2" gate="G$1" x="-139.7" y="38.1"/>
@@
 <instance part="+3V10" gate="G$1" x="-154.94" y="25.4" rot="R90"/>
 <instance part="GND14" gate="1" x="-104.14" y="58.42"/>
-<instance part="GND15" gate="1" x="-127" y="27.94"/>
-<instance part="USER_BUTTON" gate="J$1" x="-106.68" y="7.62"/>
-<instance part="GND3" gate="1" x="-99.06" y="0"/>
 <instance part="RESET_BUTTON" gate="J$1" x="-116.84" y="73.66"/>
 <instance part="GND4" gate="1" x="-104.14" y="68.58"/>
@@
 <instance part="U$3" gate="G$1" x="-7.62" y="154.94"/>
 <instance part="GND8" gate="1" x="-25.4" y="149.86"/>
+<instance part="LED3" gate="G$1" x="58.42" y="91.44" rot="R90"/>
+<instance part="GND16" gate="1" x="73.66" y="88.9"/>
+<instance part="R4" gate="G$1" x="50.8" y="91.44"/>
+<instance part="USER_BUTTON1" gate="J$1" x="60.96" y="109.22" rot="R180"/>
+<instance part="GND15" gate="1" x="40.64" y="109.22"/>
 </instances>
 <busses>
@@
 </segment>
 <segment>
-<pinref part="GND15" gate="1" pin="GND"/>
-<pinref part="R2" gate="G$1" pin="1"/>
-<wire x1="-127" y1="30.48" x2="-116.84" y2="30.48" width="0.1524" layer="91"/>
-</segment>
-<segment>
-<pinref part="GND3" gate="1" pin="GND"/>
-<pinref part="USER_BUTTON" gate="J$1" pin="1"/>
-<wire x1="-99.06" y1="2.54" x2="-99.06" y2="5.08" width="0.1524" layer="91"/>
-</segment>
-<segment>
 <pinref part="RESET_BUTTON" gate="J$1" pin="1"/>
 <pinref part="GND4" gate="1" pin="GND"/>
@@
 <wire x1="-12.7" y1="152.4" x2="-25.4" y2="152.4" width="0.1524" layer="91"/>
 <pinref part="GND8" gate="1" pin="GND"/>
+</segment>
+<segment>
+<pinref part="LED3" gate="G$1" pin="C"/>
+<pinref part="GND16" gate="1" pin="GND"/>
+<wire x1="63.5" y1="91.44" x2="73.66" y2="91.44" width="0.1524" layer="91"/>
+</segment>
+<segment>
+<pinref part="USER_BUTTON1" gate="J$1" pin="1"/>
+<pinref part="GND15" gate="1" pin="GND"/>
+<wire x1="53.34" y1="111.76" x2="40.64" y2="111.76" width="0.1524" layer="91"/>
 </segment>
 </net>
@@
 </segment>
 </net>
-<net name="N$7" class="0">
-<segment>
-<pinref part="R2" gate="G$1" pin="2"/>
-<pinref part="LED2" gate="G$1" pin="C"/>
-<wire x1="-106.68" y1="30.48" x2="-104.14" y2="30.48" width="0.1524" layer="91"/>
-</segment>
-</net>
 <net name="N$10" class="0">
 <segment>
@@
 <segment>
 <pinref part="U$2" gate="G$1" pin="11.B4"/>
-<wire x1="-91.44" y1="35.56" x2="-93.98" y2="35.56" width="0.1524" layer="91"/>
-<wire x1="-93.98" y1="35.56" x2="-93.98" y2="10.16" width="0.1524" layer="91"/>
-<pinref part="USER_BUTTON" gate="J$1" pin="3"/>
-<wire x1="-93.98" y1="10.16" x2="-99.06" y2="10.16" width="0.1524" layer="91"/>
 <pinref part="R5" gate="G$1" pin="2"/>
-<wire x1="-101.6" y1="35.56" x2="-93.98" y2="35.56" width="0.1524" layer="91"/>
-<junction x="-93.98" y="35.56"/>
+<wire x1="-101.6" y1="35.56" x2="-91.44" y2="35.56" width="0.1524" layer="91"/>
 <label x="-91.44" y="35.56" size="1.778" layer="95"/>
 </segment>
 <segment>
 <pinref part="J1" gate="G$1" pin="4"/>
-<wire x1="17.78" y1="93.98" x2="33.02" y2="93.98" width="0.1524" layer="91"/>
+<wire x1="17.78" y1="93.98" x2="45.72" y2="93.98" width="0.1524" layer="91"/>
 <label x="33.02" y="93.98" size="1.778" layer="95"/>
+<wire x1="45.72" y1="93.98" x2="45.72" y2="106.68" width="0.1524" layer="91"/>
+<wire x1="45.72" y1="106.68" x2="55.88" y2="106.68" width="0.1524" layer="91"/>
 </segment>
 </net>
@@
 <segment>
 <pinref part="J1" gate="G$1" pin="3"/>
-<wire x1="17.78" y1="91.44" x2="33.02" y2="91.44" width="0.1524" layer="91"/>
+<wire x1="17.78" y1="91.44" x2="45.72" y2="91.44" width="0.1524" layer="91"/>
 <label x="33.02" y="91.44" size="1.778" layer="95"/>
-</segment>
-<segment>
-<pinref part="LED2" gate="G$1" pin="A"/>
+<pinref part="R4" gate="G$1" pin="1"/>
+</segment>
+<segment>
 <pinref part="U$2" gate="G$1" pin="12.A4"/>
-<wire x1="-96.52" y1="30.48" x2="-91.44" y2="30.48" width="0.1524" layer="91"/>
-<label x="-91.44" y="30.48" size="1.778" layer="95"/>
+<wire x1="-91.44" y1="30.48" x2="-99.06" y2="30.48" width="0.1524" layer="91"/>
+<label x="-99.06" y="30.48" size="1.778" layer="95"/>
 </segment>
 </net>
@@
 </segment>
 </net>
+<net name="N$4" class="0">
+<segment>
+<pinref part="LED3" gate="G$1" pin="A"/>
+<pinref part="R4" gate="G$1" pin="2"/>
+</segment>
+</net>

Commit message: edit
Parts:
- removed R5: 10K, Lu_hw2:R-US_0207/10
- added R2: 10K, Lu_hw2:R-US_0207/10
- renumbered LED3 to LED2
Connections:
- net +3V3: now also R2.2; no longer R5.1
- net B4: now also R2.1, USER_BUTTON1.3; no longer R5.2
Changed lines of the file:
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@@
 <part name="GND7" library="Lu_hw2" deviceset="GND" device=""/>
 <part name="+3V2" library="Lu_hw2" deviceset="+3V3" device=""/>
-<part name="+3V3" library="Lu_hw2" deviceset="+3V3" device=""/>
-<part name="R5" library="Lu_hw2" deviceset="R-US_" device="0207/10" value="10K"/>
 <part name="RESONATOR" library="Lu_hw2" deviceset="M03" device="PTH"/>
 <part name="J1" library="Lu_hw2" deviceset="M08" device=""/>
@@
 <part name="U$3" library="Lu_hw2" deviceset="SWITCH" device=""/>
 <part name="GND8" library="Lu_hw2" deviceset="GND" device=""/>
-<part name="LED3" library="Lu_hw2" deviceset="LED" device="3MM"/>
+<part name="LED2" library="Lu_hw2" deviceset="LED" device="3MM"/>
 <part name="GND16" library="Lu_hw2" deviceset="GND" device=""/>
 <part name="R4" library="Lu_hw2" deviceset="R-US_" device="0207/10" value="330"/>
 <part name="USER_BUTTON1" library="Lu_hw2" deviceset="M03" device="PTH"/>
 <part name="GND15" library="Lu_hw2" deviceset="GND" device=""/>
+<part name="R2" library="Lu_hw2" deviceset="R-US_" device="0207/10" value="10K"/>
+<part name="+3V6" library="Lu_hw2" deviceset="+3V3" device=""/>
 </parts>
 <sheets>
@@
 <instance part="GND7" gate="1" x="-15.24" y="78.74"/>
 <instance part="+3V2" gate="G$1" x="-15.24" y="88.9" rot="R270"/>
-<instance part="+3V3" gate="G$1" x="-121.92" y="35.56" rot="R90"/>
-<instance part="R5" gate="G$1" x="-106.68" y="35.56"/>
 <instance part="RESONATOR" gate="J$1" x="-127" y="43.18"/>
 <instance part="J1" gate="G$1" x="12.7" y="93.98"/>
@@
 <instance part="U$3" gate="G$1" x="-7.62" y="154.94"/>
 <instance part="GND8" gate="1" x="-25.4" y="149.86"/>
-<instance part="LED3" gate="G$1" x="58.42" y="91.44" rot="R90"/>
+<instance part="LED2" gate="G$1" x="58.42" y="91.44" rot="R90"/>
 <instance part="GND16" gate="1" x="73.66" y="88.9"/>
 <instance part="R4" gate="G$1" x="50.8" y="91.44"/>
 <instance part="USER_BUTTON1" gate="J$1" x="60.96" y="109.22" rot="R180"/>
 <instance part="GND15" gate="1" x="40.64" y="109.22"/>
+<instance part="R2" gate="G$1" x="58.42" y="99.06"/>
+<instance part="+3V6" gate="G$1" x="71.12" y="99.06" rot="R270"/>
 </instances>
 <busses>
@@
 </segment>
 <segment>
-<pinref part="LED3" gate="G$1" pin="C"/>
+<pinref part="LED2" gate="G$1" pin="C"/>
 <pinref part="GND16" gate="1" pin="GND"/>
 <wire x1="63.5" y1="91.44" x2="73.66" y2="91.44" width="0.1524" layer="91"/>
@@
 </segment>
 <segment>
-<pinref part="+3V3" gate="G$1" pin="+3V3"/>
-<pinref part="R5" gate="G$1" pin="1"/>
-<wire x1="-119.38" y1="35.56" x2="-111.76" y2="35.56" width="0.1524" layer="91"/>
-</segment>
-<segment>
 <pinref part="J1" gate="G$1" pin="2"/>
 <pinref part="+3V4" gate="G$1" pin="+3V3"/>
 <wire x1="17.78" y1="88.9" x2="40.64" y2="88.9" width="0.1524" layer="91"/>
+</segment>
+<segment>
+<pinref part="+3V6" gate="G$1" pin="+3V3"/>
+<pinref part="R2" gate="G$1" pin="2"/>
+<wire x1="68.58" y1="99.06" x2="63.5" y2="99.06" width="0.1524" layer="91"/>
 </segment>
 </net>
@@
 <segment>
 <pinref part="U$2" gate="G$1" pin="11.B4"/>
-<pinref part="R5" gate="G$1" pin="2"/>
-<wire x1="-101.6" y1="35.56" x2="-91.44" y2="35.56" width="0.1524" layer="91"/>
-<label x="-91.44" y="35.56" size="1.778" layer="95"/>
+<wire x1="-99.06" y1="35.56" x2="-91.44" y2="35.56" width="0.1524" layer="91"/>
+<label x="-99.06" y="35.56" size="1.778" layer="95"/>
 </segment>
 <segment>
 <pinref part="J1" gate="G$1" pin="4"/>
 <wire x1="17.78" y1="93.98" x2="45.72" y2="93.98" width="0.1524" layer="91"/>
+<wire x1="45.72" y1="93.98" x2="45.72" y2="99.06" width="0.1524" layer="91"/>
+<pinref part="USER_BUTTON1" gate="J$1" pin="3"/>
+<wire x1="45.72" y1="99.06" x2="45.72" y2="106.68" width="0.1524" layer="91"/>
+<wire x1="45.72" y1="106.68" x2="53.34" y2="106.68" width="0.1524" layer="91"/>
 <label x="33.02" y="93.98" size="1.778" layer="95"/>
-<wire x1="45.72" y1="93.98" x2="45.72" y2="106.68" width="0.1524" layer="91"/>
-<wire x1="45.72" y1="106.68" x2="55.88" y2="106.68" width="0.1524" layer="91"/>
+<pinref part="R2" gate="G$1" pin="1"/>
+<wire x1="53.34" y1="99.06" x2="45.72" y2="99.06" width="0.1524" layer="91"/>
+<junction x="45.72" y="99.06"/>
 </segment>
 </net>
@@
 <net name="N$4" class="0">
 <segment>
-<pinref part="LED3" gate="G$1" pin="A"/>
+<pinref part="LED2" gate="G$1" pin="A"/>
 <pinref part="R4" gate="G$1" pin="2"/>
 </segment>

Commit message: edit
Parts:
- U$3: value SWITCH -> (none)
- renumbered RESET_BUTTON to RESET, USER_BUTTON1 to USER
Changed lines of the file:
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@@
 <part name="+3V10" library="Lu_hw2" deviceset="+3V3" device=""/>
 <part name="GND14" library="Lu_hw2" deviceset="GND" device=""/>
-<part name="RESET_BUTTON" library="Lu_hw2" deviceset="M03" device="PTH"/>
+<part name="RESET" library="Lu_hw2" deviceset="M03" device="PTH"/>
 <part name="GND4" library="Lu_hw2" deviceset="GND" device=""/>
 <part name="GND5" library="Lu_hw2" deviceset="GND" device=""/>
@@
 <part name="+3V4" library="Lu_hw2" deviceset="+3V3" device=""/>
 <part name="P+1" library="Lu_hw2" deviceset="+5V" device=""/>
-<part name="U$3" library="Lu_hw2" deviceset="SWITCH" device=""/>
 <part name="GND8" library="Lu_hw2" deviceset="GND" device=""/>
 <part name="LED2" library="Lu_hw2" deviceset="LED" device="3MM"/>
 <part name="GND16" library="Lu_hw2" deviceset="GND" device=""/>
 <part name="R4" library="Lu_hw2" deviceset="R-US_" device="0207/10" value="330"/>
-<part name="USER_BUTTON1" library="Lu_hw2" deviceset="M03" device="PTH"/>
+<part name="USER" library="Lu_hw2" deviceset="M03" device="PTH"/>
 <part name="GND15" library="Lu_hw2" deviceset="GND" device=""/>
 <part name="R2" library="Lu_hw2" deviceset="R-US_" device="0207/10" value="10K"/>
 <part name="+3V6" library="Lu_hw2" deviceset="+3V3" device=""/>
+<part name="U$3" library="Lu_hw2" deviceset="SWITCH" device=""/>
 </parts>
 <sheets>
@@
 <instance part="+3V10" gate="G$1" x="-154.94" y="25.4" rot="R90"/>
 <instance part="GND14" gate="1" x="-104.14" y="58.42"/>
-<instance part="RESET_BUTTON" gate="J$1" x="-116.84" y="73.66"/>
+<instance part="RESET" gate="J$1" x="-116.84" y="73.66"/>
 <instance part="GND4" gate="1" x="-104.14" y="68.58"/>
 <instance part="GND5" gate="1" x="-25.4" y="38.1"/>
@@
 <instance part="+3V4" gate="G$1" x="43.18" y="88.9" rot="R270"/>
 <instance part="P+1" gate="1" x="43.18" y="58.42" rot="R270"/>
-<instance part="U$3" gate="G$1" x="-7.62" y="154.94"/>
 <instance part="GND8" gate="1" x="-25.4" y="149.86"/>
 <instance part="LED2" gate="G$1" x="58.42" y="91.44" rot="R90"/>
 <instance part="GND16" gate="1" x="73.66" y="88.9"/>
 <instance part="R4" gate="G$1" x="50.8" y="91.44"/>
-<instance part="USER_BUTTON1" gate="J$1" x="60.96" y="109.22" rot="R180"/>
+<instance part="USER" gate="J$1" x="60.96" y="109.22" rot="R180"/>
 <instance part="GND15" gate="1" x="40.64" y="109.22"/>
 <instance part="R2" gate="G$1" x="58.42" y="99.06"/>
 <instance part="+3V6" gate="G$1" x="71.12" y="99.06" rot="R270"/>
+<instance part="U$3" gate="G$1" x="-2.54" y="154.94"/>
 </instances>
 <busses>
@@
 </segment>
 <segment>
-<pinref part="RESET_BUTTON" gate="J$1" pin="1"/>
+<pinref part="RESET" gate="J$1" pin="1"/>
 <pinref part="GND4" gate="1" pin="GND"/>
 <wire x1="-109.22" y1="71.12" x2="-104.14" y2="71.12" width="0.1524" layer="91"/>
@@
 </segment>
 <segment>
+<wire x1="-7.62" y1="152.4" x2="-25.4" y2="152.4" width="0.1524" layer="91"/>
+<pinref part="GND8" gate="1" pin="GND"/>
 <pinref part="U$3" gate="G$1" pin="1.GND"/>
-<wire x1="-12.7" y1="152.4" x2="-25.4" y2="152.4" width="0.1524" layer="91"/>
-<pinref part="GND8" gate="1" pin="GND"/>
 </segment>
 <segment>
@@
 </segment>
 <segment>
-<pinref part="USER_BUTTON1" gate="J$1" pin="1"/>
+<pinref part="USER" gate="J$1" pin="1"/>
 <pinref part="GND15" gate="1" pin="GND"/>
 <wire x1="53.34" y1="111.76" x2="40.64" y2="111.76" width="0.1524" layer="91"/>
@@
 <wire x1="-99.06" y1="86.36" x2="-96.52" y2="86.36" width="0.1524" layer="91"/>
 <wire x1="-96.52" y1="86.36" x2="-96.52" y2="76.2" width="0.1524" layer="91"/>
-<pinref part="RESET_BUTTON" gate="J$1" pin="3"/>
+<pinref part="RESET" gate="J$1" pin="3"/>
 <wire x1="-96.52" y1="76.2" x2="-109.22" y2="76.2" width="0.1524" layer="91"/>
 <pinref part="U$2" gate="G$1" pin="1.MCLR"/>
@@
 <wire x1="17.78" y1="93.98" x2="45.72" y2="93.98" width="0.1524" layer="91"/>
 <wire x1="45.72" y1="93.98" x2="45.72" y2="99.06" width="0.1524" layer="91"/>
-<pinref part="USER_BUTTON1" gate="J$1" pin="3"/>
+<pinref part="USER" gate="J$1" pin="3"/>
 <wire x1="45.72" y1="99.06" x2="45.72" y2="106.68" width="0.1524" layer="91"/>
 <wire x1="45.72" y1="106.68" x2="53.34" y2="106.68" width="0.1524" layer="91"/>
@@
 <wire x1="-17.78" y1="137.16" x2="-20.32" y2="137.16" width="0.1524" layer="91"/>
 <junction x="-20.32" y="137.16"/>
-<pinref part="U$3" gate="G$1" pin="3.VOUT"/>
-<wire x1="-12.7" y1="147.32" x2="-17.78" y2="147.32" width="0.1524" layer="91"/>
+<wire x1="-7.62" y1="147.32" x2="-17.78" y2="147.32" width="0.1524" layer="91"/>
 <wire x1="-17.78" y1="147.32" x2="-17.78" y2="137.16" width="0.1524" layer="91"/>
 <label x="-17.78" y="144.78" size="1.778" layer="95"/>
+<pinref part="U$3" gate="G$1" pin="3.VOUT"/>
 </segment>
 </net>
@@
 <wire x1="15.24" y1="137.16" x2="-15.24" y2="137.16" width="0.1524" layer="91"/>
 <wire x1="-15.24" y1="137.16" x2="-15.24" y2="149.86" width="0.1524" layer="91"/>
+<wire x1="-15.24" y1="149.86" x2="-7.62" y2="149.86" width="0.1524" layer="91"/>
 <pinref part="U$3" gate="G$1" pin="2.VIN"/>
-<wire x1="-15.24" y1="149.86" x2="-12.7" y2="149.86" width="0.1524" layer="91"/>
-</segment>
-</net>
+</segment>
+</net>
