File: HW2/PCB Design2/Lu_version2.brd (EAGLE design)
At the start: 50 x 50 mm, 22 parts, among them J2 USB-MB-H

Commit message: edit
Parts:
- moved LED2 8.91 mm to (15.2, 34.9)
- moved C6 5.24 mm to (34.3, 19.1)
- moved C3 4.62 mm to (40.0, 22.9)
- moved C7 3.18 mm to (37.5, 40.6)
- moved C8 2.54 mm to (41.3, 35.6)
Routing:
- net +3V3: track 0.00 -> 96.2 mm
- net +5V: track 0.00 -> 91.3 mm, vias 0 -> 2
- net B4: track 0.00 -> 90.9 mm, vias 0 -> 2
- net N$1: track 0.00 -> 78.9 mm, vias 0 -> 3
- net VSS: track 0.00 -> 64.9 mm, vias 0 -> 4
- net VDD: track 0.00 -> 51.4 mm, vias 0 -> 2
- net MCLR: track 0.00 -> 41.9 mm
- net D-: track 0.00 -> 41.0 mm, vias 0 -> 1
- net A4: track 0.00 -> 34.2 mm
- net PGD1: track 0.00 -> 29.1 mm, vias 0 -> 2
- net D+: track 0.00 -> 28.4 mm, vias 0 -> 1
- net B9: track 0.00 -> 27.8 mm
- net B8: track 0.00 -> 27.8 mm
- net B7: track 0.00 -> 27.8 mm
- net PGC1: track 0.00 -> 27.1 mm, vias 0 -> 2
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Other:
- board text added: "3V3"
- board text added: "5V"
- board text added: "A0"
- board text added: "A1"
- board text added: "A4"
- board text added: "B13"
- board text added: "B14"
- board text added: "B15"
- board text added: "B2"
- board text added: "B3"
- board text added: "B4"
- board text added: "B7"
- board text added: "B8"
- board text added: "B9"
- board text added: "D+"
- board text added: "D-"
- board text added: "GND"
- board text added: "ID"
- board text added: "Li-Chun Lu Northwestern University ME433 Advanced Mechatronics April 2016"
- board text added: "MCLR"
- board text added: "PGC1"
- board text added: "PGD1"
- board text added: "VBUS"
- board text added: "VDD"
- board text added: "VSS"
